File: Microcontroladores/Placas/Placas.kicad_pcb (KiCad board)
At the start: 2 copper layers, 39.4 x 66 mm, 18 parts

Commit message: Add Placas
Parts:
- added COMM2: CONN_01X01, Pin_Headers:Pin_Header_Straight_1x01_Pitch2.54mm, F.Cu at (81.3, 132.1)
- added COMM3: CONN_01X01, Pin_Headers:Pin_Header_Straight_1x01_Pitch2.54mm, F.Cu at (123.2, 54.6)
- added D_10: LED, LEDs:LED_D5.0mm, F.Cu at (76.2, 73.7)
- added D_11: LED, LEDs:LED_D5.0mm, F.Cu at (72.4, 44.5)
- added D_12: LED, LEDs:LED_D5.0mm, F.Cu at (66.0, 54.6)
- added D_13: LED, LEDs:LED_D5.0mm, F.Cu at (50.8, 66.0)
- added D_14: LED, LEDs:LED_D5.0mm, F.Cu at (41.9, 43.2)
- added D_15: LED, LEDs:LED_D5.0mm, F.Cu at (62.2, 68.6)
- added D_16: LED, LEDs:LED_D5.0mm, F.Cu at (52.1, 78.7)
- added D_9: LED, LEDs:LED_D5.0mm, F.Cu at (77.5, 62.2)
- added IN2: CONN_01X08, Pin_Headers:Pin_Header_Straight_1x08_Pitch2.54mm, F.Cu at (81.3, 138.4)
- added IN3: CONN_01X08, Pin_Headers:Pin_Header_Straight_1x08_Pitch2.54mm, F.Cu at (121.9, 62.2)
- added R_10: R, Resistors_THT:R_Axial_DIN0207_L6.3mm_D2.5mm_P10.16mm_Horizontal, F.Cu at (62.2, 135.9)
- added R_11: R, Resistors_THT:R_Axial_DIN0207_L6.3mm_D2.5mm_P10.16mm_Horizontal, F.Cu at (62.2, 139.7)
- added R_12: R, Resistors_THT:R_Axial_DIN0207_L6.3mm_D2.5mm_P10.16mm_Horizontal, F.Cu at (62.2, 143.5)
- added R_13: R, Resistors_THT:R_Axial_DIN0207_L6.3mm_D2.5mm_P10.16mm_Horizontal, F.Cu at (62.2, 147.3)
- added R_14: R, Resistors_THT:R_Axial_DIN0207_L6.3mm_D2.5mm_P10.16mm_Horizontal, F.Cu at (62.2, 151.1)
- added R_15: R, Resistors_THT:R_Axial_DIN0207_L6.3mm_D2.5mm_P10.16mm_Horizontal, F.Cu at (62.2, 154.9)
- added R_16: R, Resistors_THT:R_Axial_DIN0207_L6.3mm_D2.5mm_P10.16mm_Horizontal, F.Cu at (62.2, 158.8)
- added R_17: R, Resistors_THT:R_Axial_DIN0207_L6.3mm_D2.5mm_P10.16mm_Horizontal, F.Cu at (96.5, 54.6)
- added R_18: R, Resistors_THT:R_Axial_DIN0207_L6.3mm_D2.5mm_P10.16mm_Horizontal, F.Cu at (96.5, 59.7)
- added R_19: R, Resistors_THT:R_Axial_DIN0207_L6.3mm_D2.5mm_P10.16mm_Horizontal, F.Cu at (96.5, 64.8)
- added R_20: R, Resistors_THT:R_Axial_DIN0207_L6.3mm_D2.5mm_P10.16mm_Horizontal, F.Cu at (96.5, 69.8)
- added R_21: R, Resistors_THT:R_Axial_DIN0207_L6.3mm_D2.5mm_P10.16mm_Horizontal, F.Cu at (96.5, 74.9)
- added R_22: R, Resistors_THT:R_Axial_DIN0207_L6.3mm_D2.5mm_P10.16mm_Horizontal, F.Cu at (96.5, 80.0)
- added R_23: R, Resistors_THT:R_Axial_DIN0207_L6.3mm_D2.5mm_P10.16mm_Horizontal, F.Cu at (96.5, 85.1)
- added R_24: R, Resistors_THT:R_Axial_DIN0207_L6.3mm_D2.5mm_P10.16mm_Horizontal, F.Cu at (96.5, 90.2)
- added R_9: R, Resistors_THT:R_Axial_DIN0207_L6.3mm_D2.5mm_P10.16mm_Horizontal, F.Cu at (62.2, 132.1)
- added SW1: SW_DIP_x08, Buttons_Switches_THT:SW_DIP_x8_W7.62mm_Slide, F.Cu at (49.5, 135.9)
