File: Microcontroladores/Placas/Placas.sch (KiCad schematic (older format))
At the start: 18 parts

Commit message: Add Placas
Parts:
- added COMM2, COMM3: CONN_01X01, Pin_Headers:Pin_Header_Straight_1x01_Pitch2.54mm, symbol CONN_01X01
- added D_10, D_11, D_12, D_13, D_14, D_15, D_16, D_9: LED, LEDs:LED_D5.0mm, symbol LED
- added IN2, IN3: CONN_01X08, Pin_Headers:Pin_Header_Straight_1x08_Pitch2.54mm, symbol CONN_01X08
- added R_10, R_11, R_12, R_13, R_14, R_15, R_16, R_17, R_18, R_19, R_20, R_21, R_22, R_23, R_24, R_9: R, Resistors_THT:R_Axial_DIN0207_L6.3mm_D2.5mm_P10.16mm_Horizontal, symbol R
- added SW1: SW_DIP_x08, Buttons_Switches_THT:SW_DIP_x8_W7.62mm_Slide, symbol SW_DIP_x08
Connections:
- new net: D_9.1 (K), R_17.1
- new net: IN3.8 (P8), R_17.2
- new net: D_10.1 (K), R_18.1
- new net: IN3.7 (P7), R_18.2
- new net: D_11.1 (K), R_19.1
- new net: IN3.6 (P6), R_19.2
- new net: D_12.1 (K), R_20.1
- new net: IN3.5 (P5), R_20.2
- new net: D_13.1 (K), R_21.1
- new net: IN3.4 (P4), R_21.2
- new net: D_14.1 (K), R_22.1
- new net: IN3.3 (P3), R_22.2
- new net: D_15.1 (K), R_23.1
- new net: IN3.2 (P2), R_23.2
- new net: D_16.1 (K), R_24.1
- new net: IN3.1 (P1), R_24.2
- new net: COMM3.1 (P1), D_10.2 (A), D_11.2 (A), D_12.2 (A), D_13.2 (A), D_14.2 (A), D_15.2 (A), D_16.2 (A), D_9.2 (A)
- new net: IN2.1 (P1), R_9.1, SW1.16
- new net: R_10.2, R_11.2, R_12.2, R_13.2, R_14.2, R_15.2, R_16.2, R_9.2
- new net: IN2.2 (P2), R_10.1, SW1.15
- new net: IN2.8 (P8), R_16.1, SW1.9
- new net: IN2.7 (P7), R_15.1, SW1.10
- new net: IN2.6 (P6), R_14.1, SW1.11
- new net: IN2.5 (P5), R_13.1, SW1.12
- new net: IN2.4 (P4), R_12.1, SW1.13
- new net: IN2.3 (P3), R_11.1, SW1.14
- new net: COMM2.1 (P1), SW1.1, SW1.2, SW1.3, SW1.4, SW1.5, SW1.6, SW1.7, SW1.8
Other:
- note added: "Cátodo común: Activo en Alto"
- note added: "Dip switch x8"
- note added: "Ánodo Común: Activa en bajo"
- moved on the sheet: COMM1, D_1, D_2, D_3, D_4, D_5, D_6, D_7, D_8, IN1, R_1, R_2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
